File: HW/HumbuckerAmplifier.sch (KiCad schematic (older format))
At the start: 43 parts, among them J1 Conn_01x01, J10 Conn_01x01, J11 Conn_01x01, J12 Conn_01x01, J13 Conn_01x01, J14 Conn_01x01, J15 Conn_01x01, J2 Conn_01x01, J3 Conn_01x01, J4 Conn_01x01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

Commit message: Add docs & info
Parts:
- MARK1: symbol NeofoxxLibs:LOGO -> Kicad_Library:LOGO
Other:
- note added: "Both ends of the humbucker go to J3 and J4\nMiddle of buckers goes to GND (J5)"
- note added: "Output, to volume control"
- note added: "VOICING\nEffect of C3 & C4:\n- lower value == less bass\n- bigger value -> more bass\n\nEffect of (R3+R8) or (R4+R5)\nTotal resistance of (R3+R8) or (R4+R5) is what "loads" the coil.\n-> higher values will produce more "bright" sounds with more highs\n-> lower values will be more dark, even muddy if you go to low.\n--> To start, aim for a value of around 250k.\n--> Values don't have to be the sam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"
- note removed: "Both ends of the humbucker,\nand the middle of buckers goes to GND"
- moved on the sheet: H1, H2, J1, J10, J11, J15, J2, J3, J4, J5, J8, J9
